File: 9LedCluster.kicad_sch (KiCad schematic)
At the start: 43 parts, among them J1 Input, J2 Output, U1 LMR54406DBVR, U2 TLC5971RGE

Commit message: Update parts to use new NCC library symbols, but keep footprints unchanged. Delete obsolete placement file. Regenerate BOM.
Parts:
- C1, C2: symbol Device:C_Small -> NCC:a07; Category (none) -> capacitor; DigiKeyPN 490-10700-1-ND -> (none); Height (none) -> 0.5; Location (none) -> SMT bin; MPN (none) -> GRM155R71H104KE14D; Manuf Murata -> (none); Manufacturer (none) -> Murata Electronics; Mount (none) -> SMT; MouserPN 81-GRM155R71H104KE4D -> (none); PN GRM155R71H104KE14D -> (none); Package (none) -> C0402; PackageDesc Cap 0402 -> (none); PrefVendor (none) -> 2; Price10 $0.025 -> 0.025; Rating2 (none) -> C@24V>=0.039uF; Size (none) -> 1.0x0.5; Status (none) -> active; Vendor1 (none) -> Digi-Key; Vendor1PN (none) -> 490-10700-1-ND; Vendor2 (none) -> Mouser; Vendor2PN (none) -> 81-GRM155R71H104KE4D
- C3: symbol Device:C_Small -> NCC:a0B; Category (none) -> capacitor; DigiKeyPN 587-3169-1-ND -> (none); Height (none) -> 1.25; Location (none) -> SMT bin; MPN (none) -> UMK212BB7225KG-T; Manuf Taiyo Yuden -> (none); Manufacturer (none) -> Taiyo Yuden; Mount (none) -> SMT; MouserPN 963-UMK212BB7225KG-T -> (none); PN UMK212BB7225KG-T -> (none); Package (none) -> C0805; PackageDesc Cap 0805 -> (none); PrefVendor (none) -> 2; Price10 $0.438 -> 0.192; Size (none) -> 2.0x1.25; Status (none) -> active; Vendor1 (none) -> Digi-Key; Vendor1PN (none) -> 587-3169-1-ND; Vendor2 (none) -> Mouser; Vendor2PN (none) -> 963-UMK212BB7225KG-T; Vmax 24 -> (none)
- C4: symbol Device:C_Small -> NCC:a17; Category (none) -> capacitor; DigiKeyPN 490-GRM21BZ71A226ME15LCT-ND -> (none); Height (none) -> 1.25; Location (none) -> SMT bin; MPN (none) -> GRM21BZ71A226ME15L; Manuf Murata -> (none); Manufacturer (none) -> Murata Electronics; Mount (none) -> SMT; PN GRM21BZ71A226ME15L -> (none); Package (none) -> C0805; PackageDesc Cap 0805 -> (none); PrefVendor (none) -> 0; Price10 $0.18 -> 0.182; Size (none) -> 2.0x1.25; Status (none) -> active; Vendor1 (none) -> Digi-Key; Vendor1PN (none) -> 490-GRM21BZ71A226ME15LCT-ND; Vendor2 (none) -> Mouser; Vendor2PN (none) -> 81-GRM21BZ71A226ME5L; Vmax 5 -> (none)
- C5, C6, C8: symbol Device:C_Small -> NCC:a14; Category (none) -> capacitor; DigiKeyPN 399-C0402C224M4RACTUCT-ND -> (none); Height (none) -> 0.5; Location (none) -> SMT bin; MPN (none) -> C0402C224M4RACTU; Manuf KEMET -> (none); Manufacturer (none) -> KEMET; Mount (none) -> SMT; MouserPN 80-C0402C224M4RACTU -> (none); PN C0402C224M4RACTU -> (none); Package (none) -> C0402; PackageDesc Cap 0402 -> (none); PrefVendor (none) -> 2; Price10 $0.169 -> 0.169; Size (none) -> 1.0x0.5; Status (none) -> active; Vendor1 (none) -> Digi-Key; Vendor1PN (none) -> 399-C0402C224M4RACTUCT-ND; Vendor2 (none) -> Mouser; Vendor2PN (none) -> 80-C0402C224M4RACTU; Vmax 5.5 -> (none)
- C7: symbol Device:C_Small -> NCC:a09; Category (none) -> capacitor; DigiKeyPN 587-2984-1-ND -> (none); Height (none) -> 0.8; Location (none) -> SMT bin; MPN (none) -> TMK107B7105KA-T; Manuf Taiyo Yuden -> (none); Manufacturer (none) -> Taiyo Yuden; NccNum #2 -> (none); PN TMK107B7105KA-T -> (none); Package (none) -> C0603; PackageDesc Cap 0603 -> (none); PrefVendor (none) -> 2; Price10 $0.0120 -> 0.012; Rating2 (none) -> C@5V>=0.072uF; Size (none) -> 1.6x0.8; Status (none) -> active; Vendor1 (none) -> Digi-Key; Vendor1PN (none) -> 587-2984-1-ND; Vendor2 (none) -> Mouser; Vendor2PN (none) -> 963-TMK107B7105KA-T
- D1: symbol Nwc_Library:LED_AK -> NCC:p15; Category (none) -> LED; DigiKeyPN 475-GYVJLPL1.F3-KULQ-YCYK-1-350-R18CT-ND -> (none); Height (none) -> 0.85; Imax 0.06 -> (none); Location (none) -> SMT bin; MPN (none) -> GY VJLPL1.F3-KULQ-YCYK-1; Manuf ams-OSRAM -> (none); Manufacturer (none) -> ams-OSRAM; Mount (none) -> SMT; MouserPN 720-GYVL1F3KULQYCYK1 -> (none); PN GY VJLPL1.F3-KULQ-YCYK-1 -> (none); Package (none) -> LED 0505; PackageDesc LED 0505 -> (none); PrefVendor (none) -> 2; Price10 $0.748 -> 0.748; Rating2 1.4 x 1.4mm -> (none); Size (none) -> 1.4x1.4; Status (none) -> active; Vendor1 (none) -> Digi-Key; Vendor1PN (none) -> 475-GYVJLPL1.F3-KULQ-YCYK-1-350-R18CT-ND; Vendor2 (none) -> Mouser; Vendor2PN (none) -> 720-GYVL1F3KULQYCYK1; Vmax 2.93 -> (none)
- D10: symbol Device:D_Schottky_Small_Filled -> NCC:d06; Category (none) -> diode; DigiKeyPN 4878-SKM14CT-ND -> (none); Height (none) -> 1.3; Location (none) -> SMT bin; MPN (none) -> SKM14; Manuf Diotec Semiconductor -> (none); Manufacturer (none) -> Diotec Semiconductor; Mount (none) -> SMT; MouserPN 637-SKM14 -> (none); PN SKM14 -> (none); Package (none) -> SOD-123F; PackageDesc SOD-123F -> (none); PrefVendor (none) -> 0; Price10 $0.186 -> 0.186; Size (none) -> 3.7x1.8; Status (none) -> active; Vendor1 (none) -> Digi-Key; Vendor1PN (none) -> 4878-SKM14CT-ND; Vendor2 (none) -> Mouser; Vendor2PN (none) -> 637-SKM14
- D2: symbol Nwc_Library:LED_AK -> NCC:p04; Category (none) -> LED; DigiKeyPN 475-GRVJLPL1.23-KQKS-A4R2-1-350-R18CT-ND -> (none); Height (none) -> 0.85; Imax 0.06 -> (none); Location (none) -> SMT bin; MPN (none) -> GR VJLPL1.23-KQKS-A4R2-1; Manuf ams-OSRAM -> (none); Manufacturer (none) -> ams-OSRAM; Mount (none) -> SMT; MouserPN 720-GRVL123KQKSA4R21 -> (none); PN GR VJLPL1.23-KQKS-A4R2-1 -> (none); Package (none) -> LED 0505; PackageDesc LED 0505 -> (none); PrefVendor (none) -> 2; Price10 $1.04 -> 1.04; Rating2 1.4 x 1.4mm -> (none); Size (none) -> 1.4x1.4; Status (none) -> active; Vendor1 (none) -> Digi-Key; Vendor1PN (none) -> 475-GRVJLPL1.23-KQKS-A4R2-1-350-R18CT-ND; Vendor2 (none) -> Mouser; Vendor2PN (none) -> 720-GRVL123KQKSA4R21; Vmax 2.25 -> (none)
- D3: symbol Nwc_Library:LED_Thermal -> NCC:p17; Category (none) -> LED; DigiKeyPN 90-XEGAVT-H2-0000-000-000000K2001CT-ND -> (none); Height (none) -> 1; Imax 0.12 -> (none); Location (none) -> SMT bin; MPN (none) -> XEGAVT-H0-0000-000-000000K2001; Manuf Cree -> (none); Manufacturer (none) -> Cree; Mount (none) -> SMT; MouserPN 941-XEGAVTH000K2001 -> (none); PN XEGAVT-H0-0000-000-000000K2001 -> (none); Package (none) -> LED 0806; PackageDesc LED 0806 -> (none); PrefVendor (none) -> 0; Price10 $3.8190 -> 3.819; Rating2 2.05 x 1.6 mm -> (none); Size (none) -> 2.05x1.6; Status (none) -> active; Vendor1 (none) -> Digi-Key; Vendor1PN (none) -> 90-XEGAVT-H2-0000-000-000000K2001CT-ND; Vendor2 (none) -> Mouser; Vendor2PN (none) -> 941-XEGAVTH000K2001; Vmax 2.90 -> (none)
- D4: value White -> White 4000K; symbol Nwc_Library:LED_AK -> NCC:p05; Category (none) -> LED; DigiKeyPN 475-GWVJLPL1.CM-K3LX-XX55-1-350-R18CT-ND -> (none); Height (none) -> 0.85; Imax 0.06 -> (none); Location (none) -> SMT bin; MPN (none) -> GW VJLPL1.CM-K3LX-XX55-1; Manuf ams-OSRAM -> (none); Manufacturer (none) -> ams-OSRAM; Mount (none) -> SMT; MouserPN 720-GWVL1CMK3LXXX551 -> (none); PN GW VJLPL1.CM-K3LX-XX55-1 -> (none); Package (none) -> LED 0505; PackageDesc LED 0505 -> (none); PrefVendor (none) -> 1; Price10 $1.013 -> 1.013; Rating2 1.4 x 1.4mm -> (none); Size (none) -> 1.4x1.4; Status (none) -> active; Vendor1 (none) -> Digi-Key; Vendor1PN (none) -> 475-GWVJLPL1.CM-K3LX-XX55-1-350-R18CT-ND; Vendor2 (none) -> Mouser; Vendor2PN (none) -> 720-GWVL1CMK3LXXX551; Vmax 2.80 -> (none)
- D5: symbol Nwc_Library:LED_Thermal -> NCC:p18; Category (none) -> LED; DigiKeyPN 90-XEGAHR-H2-0000-000-000000H6001CT-ND -> (none); Height (none) -> 1; Imax 0.12 -> (none); Location (none) -> SMT bin; MPN (none) -> XEGAHR-H2-0000-000-000000H6001; Manuf Cree -> (none); Manufacturer (none) -> Cree; Mount (none) -> SMT; MouserPN 941-XEGAHRH200H6001 -> (none); PN XEGAHR-H2-0000-000-000000H6001 -> (none); Package (none) -> LED 0806; PackageDesc LED 0806 -> (none); PrefVendor (none) -> 0; Price10 $2.73 -> 2.73; Rating2 2.05 x 1.6 mm -> (none); Size (none) -> 2.05x1.6; Status (none) -> active; Vendor1 (none) -> Digi-Key; Vendor1PN (none) -> 90-XEGAHR-H2-0000-000-000000H6001CT-ND; Vendor2 (none) -> Mouser; Vendor2PN (none) -> 941-XEGAHRH200H6001; Vmax 2.25 -> (none)
- D6: symbol Nwc_Library:LED_Thermal -> NCC:p19; Category (none) -> LED; DigiKeyPN 90-XEGACY-H0-0000-000-000000S5001CT-ND -> (none); Height (none) -> 1; Imax 0.06 -> (none); Location (none) -> SMT bin; MPN (none) -> XEGACY-H2-0000-000-000000T3001; Manuf Cree -> (none); Manufacturer (none) -> Cree; Mount (none) -> SMT; MouserPN 941-XEGACYH20T3001 -> (none); PN XEGACY-H2-0000-000-000000T3001 -> (none); Package (none) -> LED 0806; PackageDesc LED 0806 -> (none); PrefVendor (none) -> 2; Price10 $3.00 -> 3; Rating2 2.05 x 1.6 mm -> (none); Size (none) -> 2.05x1.6; Status (none) -> active; Vendor1 (none) -> Digi-Key; Vendor1PN (none) -> 90-XEGACY-H0-0000-000-000000S5001CT-ND; Vendor2 (none) -> Mouser; Vendor2PN (none) -> 941-XEGACYH20T3001; Vmax 2.80 -> (none)
- D7: symbol Nwc_Library:LED_AK -> NCC:p03; Category (none) -> LED; DigiKeyPN 475-GTVJLPL1.13-LPLS-T3T4-1-350-R18CT-ND -> (none); Height (none) -> 0.85; Imax 0.06 -> (none); Location (none) -> SMT bin; MPN (none) -> GT VJLPL1.13-LPLS-T3T4-1; Manuf ams-OSRAM -> (none); Manufacturer (none) -> ams-OSRAM; Mount (none) -> SMT; MouserPN 720-GTVL113LPLST3T41 -> (none); PN GT VJLPL1.13-LPLS-T3T4-1 -> (none); Package (none) -> LED 0505; PackageDesc LED 0505 -> (none); PrefVendor (none) -> 2; Price10 $1.01 -> 1.01; Rating2 1.4 x 1.4mm -> (none); Size (none) -> 1.4x1.4; Status (none) -> active; Vendor1 (none) -> Digi-Key; Vendor1PN (none) -> 475-GTVJLPL1.13-LPLS-T3T4-1-350-R18CT-ND; Vendor2 (none) -> Mouser; Vendor2PN (none) -> 720-GTVL113LPLST3T41; Vmax 2.67 -> (none)
- D8: symbol Nwc_Library:LED_Thermal -> NCC:p0F; Category (none) -> LED; DigiKeyPN 1416-1913-1-ND -> (none); Height (none) -> 1.35; Imax 0.12 -> (none); Location (none) -> SMT bin; MPN (none) -> L1C1-FRD1000000000; Manuf Lumileds -> (none); Manufacturer (none) -> Lumileds; Mount (none) -> SMT; MouserPN 997-L1C1-FRD10000000 -> (none); PN L1C1-FRD1000000000 -> (none); Package (none) -> LED 0808; PackageDesc LED 0808 -> (none); PrefVendor (none) -> 2; Price10 $2.42 -> 2.42; Rating2 2.0 x 2.0mm -> (none); Size (none) -> 2.0x2.0; Status (none) -> active; Type Luxeon CZ -> Luxeon C; Vendor1 (none) -> Digi-Key; Vendor1PN (none) -> 1416-1913-1-ND; Vendor2 (none) -> Mouser; Vendor2PN (none) -> 997-L1C1-FRD10000000; Vmax 1.90 -> (none)
- D9: value Blue PC -> PC Blue; symbol Nwc_Library:LED_AK -> NCC:p16; Category (none) -> LED; DigiKeyPN 475-GBVJLPL1.F3-JRJT-BABB-1CT-ND -> (none); Height (none) -> 0.85; Imax 0.06 -> (none); Location (none) -> SMT bin; MPN (none) -> GB VJLPL1.F3-JRJT-BABB-1; Manuf ams-OSRAM -> (none); Manufacturer (none) -> ams-OSRAM; Mount (none) -> SMT; MouserPN 720-GBVL1F3JRJTBABB1 -> (none); PN GB VJLPL1.F3-JRJT-BABB-1 -> (none); Package (none) -> LED 0505; PackageDesc LED 0505 -> (none); PrefVendor (none) -> 2; Price10 $1.0240 -> 1.024; Rating2 1.4 x 1.4mm -> (none); Size (none) -> 1.4x1.4; Status (none) -> active; Vendor1 (none) -> Digi-Key; Vendor1PN (none) -> 475-GBVJLPL1.F3-JRJT-BABB-1CT-ND; Vendor2 (none) -> Mouser; Vendor2PN (none) -> 720-GBVL1F3JRJTBABB1; Vmax 2.85 -> (none)
- FB1: symbol Device:FerriteBead_Small -> NCC:n07; Category (none) -> ferrite; DigiKeyPN 490-5258-1-ND -> (none); Height (none) -> 0.8; Location (none) -> SMT bin; MPN (none) -> BLM18KG601SN1D; Manuf Murata Electronics -> (none); Manufacturer (none) -> Murata Electronics; PN BLM18KG601SN1D -> (none); Package (none) -> 0603; PackageDesc Res 0603 -> (none); PrefVendor (none) -> 1; Price10 $0.062 -> 0.062; Rating 600 Ohms @ 100MHz -> 1.3A; Rating2 1.3A -> DCR=150mΩ; Rating3 DCR=150mOhm -> (none); Size (none) -> 1.6x0.8; Status (none) -> active; Vendor1 (none) -> Digi-Key; Vendor1PN (none) -> 490-5258-1-ND
- L1: symbol Device:L_Ferrite -> NCC:n05; Category (none) -> inductor; DigiKeyPN 445-BCL322520RT-150M-DCT-ND -> (none); Height (none) -> 2; Location (none) -> SMT bin; MPN (none) -> BCL322520RT-150M-D; Manuf TDK -> (none); Manufacturer (none) -> TDK; Mount (none) -> SMT; MouserPN 810-BCL322520RT150MD -> (none); PN BCL322520RT-150M-D -> (none); Package (none) -> Ind 3.2x2.5mm; PackageDesc Ind 1210 -> (none); PrefVendor (none) -> 2; Price10 $1.09 -> 1.09; Rating I=1.47, Isat=1.33 -> I=1.47; Rating2 DCR=0.32 -> 320 mOhm Max; Size (none) -> 3.2x2.5; Status (none) -> active; Tolerance (none) -> 20%; Vendor1 (none) -> Digi-Key; Vendor1PN (none) -> 445-BCL322520RT-150M-DCT-ND; Vendor2 (none) -> Mouser; Vendor2PN (none) -> 810-BCL322520RT150MD
- R1: symbol Device:R_Small_US -> NCC:r22; Category (none) -> resistor; DigiKeyPN RR08P24.9KDCT-ND -> (none); Height (none) -> 0.4; Location (none) -> SMT bin; MPN (none) -> RR0816P-2492-D-39C; Manuf Susumu -> (none); Manufacturer (none) -> Susumu; Mount (none) -> SMT; MouserPN 754-RR0816P-2492D39C -> (none); PN RR0816P-2492-D-39C -> (none); Package (none) -> R0603; PackageDesc Res 0603 -> (none); PrefVendor (none) -> 0; Price10 $0.025 -> 0.025; Rating2 (none) -> 25ppm/C; Size (none) -> 1.6x0.8; Status (none) -> active; Vendor1 (none) -> Digi-Key; Vendor1PN (none) -> RR08P24.9KDCT-ND; Vendor2 (none) -> Mouser; Vendor2PN (none) -> 754-RR0816P-2492D39C; Vmax 4.0 -> (none)
- R2: symbol Device:R_Small_US -> NCC:r1B; Category (none) -> resistor; DigiKeyPN 2019-RK73Z1ETTPCT-ND -> (none); Height (none) -> 0.35; Imax 0.6 -> (none); Location (none) -> SMT bin; MPN (none) -> RK73Z1ETTP; Manuf KOA Speer -> (none); Manufacturer (none) -> KOA Speer; Mount (none) -> SMT; MouserPN 660-RK73Z1ETTP -> (none); PN RK73Z1ETTP -> (none); Package (none) -> R0402; PackageDesc Res 0402 -> (none); Pmax 0.0 -> (none); PrefVendor (none) -> 2; Price10 $0.008 -> 0.008; Rating2 1A -> (none); Size (none) -> 1.0x0.5; Status (none) -> active; Vendor1 (none) -> Digi-Key; Vendor1PN (none) -> 2019-RK73Z1ETTPCT-ND; Vendor2 (none) -> Mouser; Vendor2PN (none) -> 660-RK73Z1ETTP; Vmax 0.0 -> (none)
- R3: symbol Device:R_Small_US -> NCC:r14; Category (none) -> resistor; DigiKeyPN 311-100KDCT-ND -> (none); Height (none) -> 0.45; Imax 0.00003 -> (none); Location (none) -> SMT bin; MPN (none) -> RT0603DRD07100KL; Manuf YAGEO -> (none); Manufacturer (none) -> YAGEO; Mount (none) -> SMT; MouserPN 603-RT0603DRD07100KL -> (none); PN RT0603DRD07100KL -> (none); Package (none) -> R0603; PackageDesc Res 0603 -> (none); Pmax 0.00013 -> (none); PrefVendor (none) -> 2; Price10 $0.048 -> 0.048; Rating2 (none) -> 25ppm/C; Size (none) -> 1.6x0.8; Status (none) -> active; Vendor1 (none) -> Digi-Key; Vendor1PN (none) -> 311-100KDCT-ND; Vendor2 (none) -> Mouser; Vendor2PN (none) -> 603-RT0603DRD07100KL; Vmax 1 -> (none)
- R4, R5: symbol Device:R_Small_US -> NCC:r1C; Category (none) -> resistor; DigiKeyPN YAG3343CT-ND -> (none); Height (none) -> 0.2; Imax 0.0015 -> (none); Location (none) -> SMT bin; MPN (none) -> RT0402FRE0727RL; Manuf YAGEO -> (none); Manufacturer (none) -> YAGEO; Mount (none) -> SMT; MouserPN 603-RT0402FRE0727RL -> (none); PN RT0402FRE0727RL -> (none); Package (none) -> R0402; PackageDesc Res 0402 -> (none); Pmax 0.0019 -> (none); PrefVendor (none) -> 2; Price10 $0.021 -> 0.021; Rating2 (none) -> 50ppm/C; Size (none) -> 1.0x0.5; Status (none) -> active; Vendor1 (none) -> Digi-Key; Vendor1PN (none) -> YAG3343CT-ND; Vendor2 (none) -> Mouser; Vendor2PN (none) -> 603-RT0402FRE0727RL; Vmax 1.24 -> (none)
- R6: symbol Device:R_Small_US -> NCC:r25; Category (none) -> resistor; DigiKeyPN 2019-RK73H1JTTD10R0FCT-ND -> (none); Height (none) -> 0.45; Location (none) -> SMT bin; MPN (none) -> RK73H1JTTD10R0F; Manuf KOA Speer -> (none); Manufacturer (none) -> KOA Speer; Mount (none) -> SMT; MouserPN 660-RK73H1JTTD10R0F -> (none); PN RK73H1JTTD10R0F -> (none); Package (none) -> R0603; PackageDesc Res 0603 -> (none); PrefVendor (none) -> 0; Price10 $0.016 -> 0.016; Rating2 (none) -> 100ppm/C; Size (none) -> 1.6x0.8; Status (none) -> active; Vendor1 (none) -> Digi-Key; Vendor1PN (none) -> 2019-RK73H1JTTD10R0FCT-ND; Vendor2 (none) -> Mouser; Vendor2PN (none) -> 660-RK73H1JTTD10R0F
- R7: symbol Device:R_Small_US -> NCC:r0B; Category (none) -> resistor; DigiKeyPN 408-RR0510P-8250-DCT-ND -> (none); Height (none) -> 0.35; Imax 0.0015 -> (none); Location (none) -> SMT bin; MPN (none) -> RR0510P-8250-D; Manuf Susumu -> (none); Manufacturer (none) -> Susumu; Mount (none) -> SMT; MouserPN 754-RR0510P-8250D -> (none); PN RR0510P-8250-D -> (none); Package (none) -> R0402; PackageDesc Res 0402 -> (none); Pmax 0.0019 -> (none); PrefVendor (none) -> 2; Price10 $0.024 -> 0.024; Rating2 (none) -> 25ppm/C; Size (none) -> 1.0x0.5; Status (none) -> active; Vendor1 (none) -> Digi-Key; Vendor1PN (none) -> 408-RR0510P-8250-DCT-ND; Vendor2 (none) -> Mouser; Vendor2PN (none) -> 754-RR0510P-8250D; Vmax 1.24 -> (none)
- R8, R9: symbol Device:R_Small_US -> NCC:r26; Category (none) -> resistor; DigiKeyPN 2019-RK73H1JTTD12R0FCT-ND -> (none); Height (none) -> 0.45; Location (none) -> SMT bin; MPN (none) -> RK73H1JTTD12R0F; Manuf KOA Speer -> (none); Manufacturer (none) -> KOA Speer; Mount (none) -> SMT; MouserPN 660-RK73H1JTTD12R0F -> (none); PN RK73H1JTTD12R0F -> (none); Package (none) -> R0603; PackageDesc Res 0603 -> (none); PrefVendor (none) -> 0; Price10 $0.026 -> 0.026; Rating2 (none) -> 100ppm/C; Size (none) -> 1.6x0.8; Status (none) -> active; Vendor1 (none) -> Digi-Key; Vendor1PN (none) -> 2019-RK73H1JTTD12R0FCT-ND; Vendor2 (none) -> Mouser; Vendor2PN (none) -> 660-RK73H1JTTD12R0F
- U1: value LMR54406DBVR -> LMR54406; symbol Nwc_Library:LMR54406 -> NCC:k16; Category (none) -> IC; DigiKeyPN 296-LMR54406DBVRCT-ND -> (none); Height (none) -> 1.2; Location (none) -> SMT bin; MPN (none) -> LMR54406DBVR; Manuf TI -> (none); Manufacturer (none) -> TI; Mount (none) -> SMT; MouserPN 595-LMR54406DBVR -> (none); PN LMR54406DBVR -> (none); Package (none) -> SOT-23-6; PackageDesc SOT-23-6 -> (none); PrefVendor (none) -> 2; Price10 $0.86 -> 0.86; Size (none) -> 2.9x2.8; Status (none) -> active; Type Step down -> Regulator, Buck; Vendor1 (none) -> Digi-Key; Vendor1PN (none) -> 296-LMR54406DBVRCT-ND; Vendor2 (none) -> Mouser; Vendor2PN (none) -> 595-LMR54406DBVR
- U2: value TLC5971RGE -> TLC5971; symbol Driver_LED:TLC5971RGE -> NCC:k05; Category (none) -> IC; DigiKeyPN 296-28448-1-ND -> (none); Height (none) -> 1; Location (none) -> SMT bin; MPN (none) -> TLC5971RGER; Manuf TI -> (none); Manufacturer (none) -> TI; Mount (none) -> SMT; MouserPN 595-TLC5971RGER -> (none); PN TLC5971RGER -> (none); Package (none) -> VQFN-24 4x4mm_P0.5mm; PackageDesc VQFN-24 4x4mm_P0.5mm -> (none); PrefVendor (none) -> 0; Price10 $2.34 -> 2.342; Rating2 (none) -> 12ch, 16bit; Size (none) -> 4.0x4.0; Status (none) -> active; Vendor1 (none) -> Digi-Key; Vendor1PN (none) -> 296-28448-1-ND; Vendor2 (none) -> Mouser; Vendor2PN (none) -> 595-TLC5971RGER; Vmax 5.5 -> (none)
- Z1, Z2, Z3, Z4: value 5V -> 5.5V; symbol Diode:5KPxxCA -> NCC:d04; Category (none) -> diode; DigiKeyPN 478-10594-1-ND -> (none); Height (none) -> 0.5; Location (none) -> SMT bin; MPN (none) -> GG040205100N2P; Manuf KYOCERA AVX -> (none); Manufacturer (none) -> KYOCERA AVX; Mount (none) -> SMT; MouserPN 581-GG040205100N2P -> (none); PN GG040205100N2P -> (none); Package (none) -> TVS-0402; PackageDesc Res 0402 -> (none); PrefVendor (none) -> 2; Price10 $0.127 -> 0.127; Rating 10 pF -> 5.5V, 10pF; Size (none) -> 1.0x0.6; Status (none) -> active; Vendor1 (none) -> Digi-Key; Vendor1PN (none) -> 478-10594-1-ND; Vendor2 (none) -> Mouser; Vendor2PN (none) -> 581-GG040205100N2P
